Commit message: pt_mujoco: use the BAM-identified STS3215 profile for the pan and tilt servos
Adds sts3215.mjcf.xacro (class pt_sts3215, distinct from lekiwi's sts3215 so both can be composed)
and applies its gain, damping, armature and friction at build time like the wheels. The step
response settles in about 0.3 s with 4% (pan) to 8% (tilt) overshoot instead of 0.55 s with none.

Co-Authored-By: Claude Sonnet 5 <noreply@anthropic.com>

File: pt_mujoco/mjcf/pantilt.mjcf.xacro (robot description, xacro)
@@ -62,5 +62,5 @@
         <inertial pos="-9.07886e-05 0.0590972 -0.0172669" mass="0.119226"
                   diaginertia="5.94278e-05 5.89975e-05 3.13712e-05"/>
-        <joint name="shoulder_pan_joint" class="pan"/>
+        <joint name="shoulder_pan_joint" class="pt_sts3215" axis="0 0 1" range="-1.5708 1.5708"/>
         <geom mesh="shoulder_link_mesh" material="light_grey" class="visual"
               pos="${shoulder_link_geom_pos}" quat="${shoulder_link_geom_quat}"/>
