Commit message: Trim comments and docstrings to one line, refresh package.xml files, drop test_without_ros
Co-Authored-By: Claude Sonnet 5 <noreply@anthropic.com>

File: pt_description/urdf/oakd_s2.module.xacro (robot description, xacro)
@@ -2,8 +2,5 @@
 <robot name="depthai_camera"
 	xmlns:xacro="http://ros.org/wiki/xacro">
-	<!--
-	  Custom OAK-D-S2 camera macro, shared by both pt100/pt101.
-	  This version allows direct color parameterization (r/g/b/a) for the mesh material.
-	-->
+	<!-- OAK-D S2 camera macro shared by pt100/pt101, with r/g/b/a mesh colour parameters -->
 	<xacro:macro name="oakd_s2_camera"
 		params="camera_name parent base_frame

File: pt_description/urdf/pantilt.common.xacro (robot description, xacro)
@@ -5,10 +5,5 @@
   <xacro:property name="charcoal_rgba" value="0.15 0.15 0.15 1.0"/>
   <xacro:property name="charcoal_rgb" value="0.15"/>
-  <!-- Pan-tilt mechanical configuration: selects pantilt_base / shoulder_pan mesh
-       variants. "pt101" (default, recommended) uses the SO-ARM101-based
-       meshes; "pt100" uses the original SO-ARM100-based meshes. All
-       link/joint origins, axes, and the mount to the host robot are shared
-       and unchanged across configs — pt101 is a drop-in mesh replacement
-       only. -->
+  <!-- Mesh variant: pt101 (default, recommended) or pt100; only the meshes differ, all origins and axes are shared -->
   <xacro:arg name="pantilt_config" default="pt101"/>
   <xacro:property name="pantilt_config" value="$(arg pantilt_config)"/>
@@ -20,11 +15,5 @@
   <xacro:property name="pantilt_base_mesh" value="pantilt_base_100.stl"/>
   <xacro:property name="shoulder_pan_mesh" value="pan_joint_100.stl"/>
-  <!-- Mesh-local origin correction, applied to the body mesh of each link
-       only (not the motor meshes), in place of the shared
-       pantilt_offset_rz / shoulder_offset_rx+rz rotations above. pt100 meshes
-       reuse those shared rotations with zero translation (no-op). pt101
-       meshes need a different rotation (SO-ARM101's base_link/shoulder_link
-       frames are not simply Z-rotated copies of SO-ARM100's) plus a
-       translation; see derivation below. -->
+  <!-- Mesh-local origin correction for the body meshes only; pt100 reuses the shared rotations, pt101 needs its own -->
   <xacro:property name="pantilt_base_mesh_rpy" value="0 0 ${pantilt_offset_rz}"/>
   <xacro:property name="shoulder_pan_mesh_rpy" value="${shoulder_offset_rx} 0 ${shoulder_offset_rz}"/>
@@ -39,24 +28,13 @@
     <xacro:property name="shoulder_pan_mesh_xyz" value="-0.0120 0 -0.0463059"/>
   </xacro:if>
-  <!-- Shoulder-pan joint origin (in reoriented base_link frame). Z is offset +0.0483559 from
-       the raw SO100-derived value (0.0165) so shoulder_pan_joint's origin sits relative to
-       shoulder_link's own mesh the same way SO101's shoulder_pan_joint sits relative to
-       shoulder_link (mesh-bbox-vs-origin alignment verified against so101.urdf);
-       shoulder_pan_mesh_xyz and tilt_motor's mesh offset above/below carry the
-       equal-and-opposite compensation so no visual or downstream frame (tilt_joint,
-       tilt_link, oak_link) moves. -->
+  <!-- Shoulder-pan joint origin; z is offset from the SO100 value and compensated in the mesh and tilt offsets so no frame moves -->
   <xacro:property name="shoulder_pan_x" value="0.0452"/>
   <xacro:property name="shoulder_pan_z" value="0.0648559"/>
-  <!-- Joint limits - single source of truth for pantilt.module.xacro's URDF <limit> elements
-       (needed as globals here, not macro params, since pantilt.module.xacro always includes
-       this file directly - see pantilt.joints.xacro's own matching defaults, used separately
-       for its ros2_control <joint> blocks). -->
+  <!-- Joint limits for the URDF <limit> elements (pantilt.joints.xacro has matching defaults for ros2_control) -->
   <xacro:property name="shoulder_pan_lower" value="-1.5708"/>
   <xacro:property name="shoulder_pan_upper" value="1.5708"/>
   <xacro:property name="tilt_joint_lower" value="-1.5708"/>
   <xacro:property name="tilt_joint_upper" value="1.5708"/>
-  <!-- Tilt joint origin (in shoulder_link frame — same as SO100 shoulder_lift, minus the same
-       -0.0483559 compensation applied to shoulder_pan_z above, so shoulder_pan_z + tilt_joint_z
-       — and therefore tilt_link's world pose — is unchanged). -->
+  <!-- Tilt joint origin in shoulder_link; the z offset cancels the shoulder_pan_z compensation above -->
   <xacro:property name="tilt_joint_x" value="0.0306"/>
   <xacro:property name="tilt_joint_z" value="0.0541441"/>

File: pt_description/urdf/pantilt.control.xacro (robot description, xacro)
@@ -8,32 +8,16 @@
   <xacro:arg name="sts3215_max_vel_steps" default="3400"/>   <!-- STS3215=3400, STS3032=2900, STS3235=3400 -->
   <xacro:arg name="proportional_vel_max"   default="0"/>      <!-- [0-max_velocity_steps]; 0 = each joint uses commanded velocity -->
-  <!-- Servo EEPROM profile (0-254 each, written per joint at start-up). Defaults match
-       pantilt.joints.xacro's macro defaults (the slow, smooth profile); pt_control's
-       urdf_config.yaml sets them explicitly so they can be tuned without editing xacro. -->
+  <!-- Servo EEPROM profile (0-254), defaults match pantilt.joints.xacro; urdf_config.yaml sets them for tuning -->
   <xacro:arg name="internal_max_vel"       default="65"/>
   <xacro:arg name="internal_max_acc"       default="50"/>
   <xacro:arg name="internal_acc_coeff"     default="0"/>
-  <!-- Motor IDs, step-centering, and joint limits are NOT xacro:args here - they're
-       physical-calibration constants for this mechanism (motor wiring, servo centering),
-       not per-deployment connection settings, so pantilt.joints.xacro's macro defaults are
-       their single source of truth (same convention as so101.control.xacro/so100.control.xacro
-       in so_arm_ros2, which hardcode motor IDs/joint limits as fixed xacro:property values
-       rather than sourcing them from an external launch-time YAML). A host embedding this
-       mechanism on a shared bus (e.g. lekiwi_ros2's base_pantilt.control.xacro) can still
-       override any of pantilt_joints' macro params explicitly if it ever needs different
-       values - see pantilt.joints.xacro. -->
+  <!-- Motor IDs, centres and joint limits are calibration constants: pantilt.joints.xacro macro defaults hold them -->
   <!-- Simulation -->
-  <!-- "real" (default) keeps the STS3215 serial hardware plugin below unchanged.
-       "gazebo" swaps the <hardware> plugin for gz_ros2_control/GazeboSimSystem.
-       "mujoco" swaps it for mujoco_ros2_control/MujocoSystemInterface.
-       Both implement the same SystemInterface contract - the joints and controllers stay
-       identical in all three cases. -->
+  <!-- Hardware plugin: real (STS3215, default), gazebo or mujoco; joints and controllers are identical -->
   <xacro:arg name="ros2_control_hardware_type" default="real"/>
   <!-- Path to the controllers YAML the embedded controller_manager should load; only
        used when the <gazebo> plugin below is actually instantiated (i.e. in sim). -->
   <xacro:arg name="simulation_controllers" default=""/>
-  <!-- mujoco mode only: path to the MJCF generated by pt_mujoco's build_mujoco_models (see
-       pt_control/launch/pantilt.launch.py; pantilt_config picks the pt100/pt101 variant) and
-       whether to open the MuJoCo Simulate viewer window. -->
+  <!-- mujoco only: generated MJCF path and whether to open the viewer -->
   <xacro:arg name="mujoco_model" default=""/>
   <xacro:arg name="mujoco_headless" default="false"/>
@@ -41,12 +25,6 @@
        because pantilt_joints (called below) writes it per joint as max_velocity_steps. -->
   <xacro:property name="sts3215_max_vel_steps" value="$(arg sts3215_max_vel_steps)"/>
-  <!-- Torque limit as a top-level property — required by pantilt.module.xacro for the URDF
-       <limit> elements on the revolute joints.
-       pantilt_max_velocity_rads duplicates pantilt_joints' own local computation
-       (pantilt.joints.xacro) - only used by module.xacro's gazebo-mode <limit velocity>,
-       real and mujoco modes keep velocity="1e6" (see module.xacro's comment on why) regardless. -->
-  <!-- This project runs the 12V STS3215 variant: 30 kgf*cm stall torque per Feetech's
-       datasheet for that voltage option (not the 7.4V/19.5 kgf*cm variant used by stock
-       SO-ARM100/101). -->
+  <!-- Torque limit for the module's revolute joint <limit> elements -->
+  <!-- 12V STS3215: 30 kgf*cm stall torque -->
   <xacro:property name="max_torque_nm"    value="2.942"/>  <!-- N⋅m (30 kgf⋅cm @ 12V) -->
   <xacro:property name="pantilt_max_velocity_steps" value="${int(sts3215_max_vel_steps * 0.85)}"/>

File: pt_description/urdf/pantilt.joints.xacro (robot description, xacro)
@@ -1,25 +1,5 @@
 <?xml version="1.0"?>
 <robot xmlns:xacro="http://www.ros.org/wiki/xacro">
-  <!--
-    pantilt_joints macro — ros2_control joint declarations for the PT100 pan-tilt.
-    Intended for embedding into a host robot's <ros2_control> block when the
-    PT100 shares the host's serial bus (and therefore its hardware interface).
-    For standalone use, pantilt.control.xacro wraps this in its own <ros2_control>
-    block with the STSHardwareInterface plugin.
-    Params:
-      shoulder_pan_motor_id — STS3215 motor ID for pan axis
-      tilt_motor_id         — STS3215 motor ID for tilt axis
-      shoulder_pan_center_steps — raw step value (0–4095) for pan centre position
-      tilt_center_steps     — raw step value (0–4095) for tilt centre position
-      sts3215_max_vel_steps — motor's max velocity in steps/s, model-dependent;
-                               written per joint as max_velocity_steps
-      internal_max_vel      — EEPROM VMax cap (addr 84), written per joint
-      internal_max_acc      — EEPROM AMax cap (addr 85), written per joint
-      internal_acc_coeff    — EEPROM KAcc coefficient (addr 86), written per joint
-      The internal_* defaults (65/50/0, near the STS3215 firmware's own ~68/~50/1) give the slow,
-      smooth motion this mechanism is meant to have. They are the module's own tuning, not a
-      per-host setting: the wheels' 254/254/100 makes the pan-tilt accelerate fast enough to draw
-      the current that crashed the Pi. A host may still pass different values to this macro.
-  -->
+  <!-- pantilt_joints: ros2_control joints for a host's shared-bus block; defaults are the mechanism's calibration and the slow 65/50/0 servo profile -->
   <xacro:macro name="pantilt_joints" params="
       shoulder_pan_motor_id:=1
@@ -56,7 +36,5 @@
       <state_interface name="velocity"/>
       <state_interface name="effort"/>
-      <!-- Real-hardware-only telemetry: neither gz_ros2_control/GazeboSimSystem nor
-           mujoco_ros2_control/MujocoSystemInterface know position/velocity/effort-only
-           joints, and simulated joints have no real telemetry for these. -->
+      <!-- Real hardware only: sim joints have no such telemetry -->
       <xacro:if value="${ros2_control_hardware_type == 'real'}">
         <state_interface name="voltage"/>
@@ -83,7 +61,5 @@
       <state_interface name="velocity"/>
       <state_interface name="effort"/>
-      <!-- Real-hardware-only telemetry: neither gz_ros2_control/GazeboSimSystem nor
-           mujoco_ros2_control/MujocoSystemInterface know position/velocity/effort-only
-           joints, and simulated joints have no real telemetry for these. -->
+      <!-- Real hardware only: sim joints have no such telemetry -->
       <xacro:if value="${ros2_control_hardware_type == 'real'}">
         <state_interface name="voltage"/>

File: pt_description/urdf/pantilt.module.xacro (robot description, xacro)
@@ -94,9 +94,5 @@
       </collision>
     </link>
-    <!-- real and mujoco modes: velocity="1e6" (unreachable) disables JointSaturationLimiter's
-         clipping, since joy_teleop's absolute position jumps would otherwise trip spurious limit
-         errors (MuJoCo does not need the limit: its servo model already bounds the motion).
-         gazebo mode: uses the real computed ceiling instead, since GazeboSimSystem actually
-         enforces this limit on the simulated joint. -->
+    <!-- real/mujoco: 1e6 avoids spurious limit trips on joystick jumps; gazebo enforces the real ceiling -->
     <!-- Shoulder-pan joint (revolute; was "pan_joint") -->
     <joint name="shoulder_pan_joint" type="revolute">

File: pt_description/urdf/pantilt.urdf.xacro (robot description, xacro)
@@ -13,7 +13,5 @@
 	  <origin xyz="0 0 0" rpy="0 0 0"/>
 	</xacro:pantilt_module>
-  <!-- Gazebo simulation: spawns controller_manager inside the gz_sim process, loading
-       $(arg simulation_controllers). Inert (ignored) outside Gazebo, so this is safe to
-       leave in place regardless of ros2_control_hardware_type. -->
+  <!-- Gazebo only: spawns controller_manager in gz_sim; inert elsewhere -->
   <gazebo>
     <plugin filename="gz_ros2_control-system" name="gz_ros2_control::GazeboSimROS2ControlPlugin">

File: pt_mujoco/mjcf/pantilt.mjcf.xacro (robot description, xacro)
@@ -1,7 +1,4 @@
 <?xml version="1.0"?>
-<!-- Parametric PT100/PT101 MJCF library (mujoco_ros2_control equivalent of pantilt.module.xacro):
-     defines the pantilt_body macro, selected by pantilt_config. pt.mjcf.xacro fixes it to the
-     world for standalone use; scenes come from mjcf/scenes and are composed by
-     build_mujoco_models.py, which also syncs the numbers below from the URDF. -->
+<!-- Parametric PT100/PT101 MJCF (pantilt_body macro, selected by pantilt_config); build_mujoco_models.py syncs the numbers from the URDF -->
 <mujoco xmlns:xacro="http://www.ros.org/wiki/xacro" model="pantilt">
   <xacro:arg name="pantilt_config" default="pt101"/>
@@ -10,10 +7,5 @@
        which only xacro resolves. -->
   <xacro:include filename="$(find pt_mujoco)/mjcf/pantilt_shared.xml"/>
-  <!-- Mesh files and mesh-local offset corrections - pt100 defaults below, overridden for
-       pt101. Not $(find)-included from pantilt.common.xacro's equivalent properties: URDF's
-       rpy composes as Rz*Ry*Rx (fixed-axis roll,pitch,yaw) while MuJoCo's default euler="xyz"
-       composes as Rx*Ry*Rz - the reverse order. These only agree when rpy has a single nonzero
-       axis; every offset below has 2+ nonzero axes, so each is given as a quat computed
-       directly from the URDF's rpy (via its own Rz*Ry*Rx convention), not a ported euler. -->
+  <!-- Mesh files and offset corrections (pt100 defaults, overridden for pt101), as quats since URDF rpy order differs from MuJoCo euler -->
   <xacro:property name="pantilt_base_mesh" value="pantilt_base_100.stl"/>
   <xacro:property name="shoulder_link_mesh_file" value="pan_joint_100.stl"/>
@@ -22,8 +14,5 @@
        pt101's) - quat is Rz(90) alone, not pt101's override value below. -->
   <xacro:property name="pantilt_base_geom_quat" value="0.70710678 0 0 0.70710678"/>
-  <!-- shoulder_link_geom_pos Z carries the same -0.0483559 reslice compensation as
-       pantilt.common.xacro's shoulder_pan_mesh_xyz (URDF side) - see that file's comment
-       for the derivation. Applies to both configs; only X differs (pt101's bracket mesh
-       has a nonzero local X offset, pt100's doesn't). -->
+  <!-- shoulder_link_geom_pos Z carries the same reslice compensation as pantilt.common.xacro; only X differs between configs -->
   <xacro:property name="shoulder_link_geom_pos" value="0 0 -0.0483559"/>
   <xacro:property name="shoulder_link_geom_quat" value="0.5 0.5 0.5 0.5"/>
@@ -40,7 +29,5 @@
     <mesh name="shoulder_link_mesh" file="$(find pt_description)/meshes/${shoulder_link_mesh_file}"/>
   </asset>
-  <!-- pantilt_base_link has no pos/euler of its own - it inherits the invocation site's
-       frame. Collision geoms cover only the primary body mesh, not the decorative "_motor"
-       sub-meshes. -->
+  <!-- pantilt_base_link inherits the invocation frame; collision geoms cover the main body mesh only -->
   <xacro:macro name="pantilt_body">
     <body name="pantilt_base_link">
@@ -48,15 +35,10 @@
       <geom mesh="pantilt_base_link_mesh" material="light_grey" class="visual"
             pos="${pantilt_base_geom_pos}" quat="${pantilt_base_geom_quat}"/>
-      <!-- quat, not euler: MuJoCo auto-aligns every mesh geom to its own principal-inertia
-           frame at compile time and composes that correction differently (and wrongly) with
-           an explicit euler= than with an explicit quat= - verified empirically per-mesh,
-           same class of bug as lekiwi_description's ld06_lidar fix. -->
+      <!-- quat, not euler: MuJoCo composes euler wrongly with a mesh's auto-aligned inertia frame -->
       <geom mesh="pan_motor" material="charcoal" class="visual"
             pos="0 0 0" quat="0.70710678 0 0 0.70710678"/>
       <geom mesh="pantilt_base_link_mesh" class="collision"
             pos="${pantilt_base_geom_pos}" quat="${pantilt_base_geom_quat}"/>
-      <!-- pos Z = 0.0648559 (was 0.0165): same reslice as pantilt.common.xacro's
-           shoulder_pan_z (URDF side) - the joint origin moved along its own rotation axis,
-           compensated by the mesh offsets above/below so nothing renders differently. -->
+      <!-- pos Z 0.0648559: same reslice as pantilt.common.xacro, compensated by the mesh offsets -->
       <body name="shoulder_link" pos="0.0452 0 0.0648559">
         <inertial pos="-9.07886e-05 0.0590972 -0.0172669" mass="0.119226"

File: pt_mujoco/mjcf/pt.mjcf.xacro (robot description, xacro)
@@ -1,7 +1,4 @@
 <?xml version="1.0"?>
-<!-- Pan-tilt payload MJCF entry point (mujoco_ros2_control equivalent of pt_description's
-     pantilt.urdf.xacro): the pantilt_body macro from pantilt.mjcf.xacro fixed to the world
-     origin, robot only. build_mujoco_models.py composes a separate scene (mjcf/scenes) and
-     syncs frames, meshes, inertias and limits from the URDF. -->
+<!-- Payload MJCF entry point: pantilt_body fixed to the world origin, robot only -->
 <mujoco xmlns:xacro="http://www.ros.org/wiki/xacro" model="pantilt">
   <xacro:arg name="pantilt_config" default="pt101"/>

File: pt_mujoco/mjcf/sts3215.mjcf.xacro (robot description, xacro)
@@ -1,19 +1,8 @@
 <?xml version="1.0"?>
-<!-- STS3215 MuJoCo joint defaults, used by the pan and tilt joints and actuators. Copied verbatim
-     from so_arm_ros2/so_arm_mujoco/mjcf/sts3215.mjcf.xacro (lekiwi_mujoco keeps its own copy for its
-     wheels, under the class name sts3215, so this one is named pt_sts3215: default class names are global
-     and would collide when the payload is attached to it) - the BAM identification is a property of the motor, not the mechanism it drives. -->
+<!-- STS3215 joint defaults for pan/tilt; class is pt_sts3215 because default class names are global and lekiwi_mujoco has sts3215 -->
 <mujoco xmlns:xacro="http://www.ros.org/wiki/xacro">
   <default class="pt_sts3215">
-    <!-- Identified from real STS3215 (12V) trajectories via Rhoban's BAM project
-         (github.com/Rhoban/bam), model "m1", params/feetech_sts3215_12V/m1.json (PR #5).
-         Derived with bam.to_mujoco's own voltage_controlled_to_mujoco formula, corrected to
-         fold in error_gain_ratio (the per-unit gain correction STS3215Actuator.compute_control
-         actually applies - bam.to_mujoco's static export omits it, a known gap in that
-         deprecated tool). kp/error_gain/max_pwm=32/0.166/0.97 are STS3215Actuator's firmware
-         constants (fixed across supply voltages); vin=12 for this identified variant. -->
-    <!-- solreflimit/solimplimit: stiff end stops. With MuJoCo's default soft limit a full-speed jump to
-         a limit penetrates it by ~0.01 rad, and ros2_control's limiter treats a measured position
-         beyond the URDF limit as a hardware fault and deactivates the controller. -->
+    <!-- BAM-identified from a real STS3215 (12V), model m1 (github.com/Rhoban/bam), with error_gain_ratio folded in -->
+    <!-- Stiff end stops: a soft limit lets a full-speed jump pass the URDF limit and deactivates the controller -->
     <joint damping="1.057835" frictionloss="0.195871" armature="0.032460"
            solreflimit="0.004 1" solimplimit="0.99 0.999 0.001 0.5 2"/>
