Commit message: Run the pan-tilt sim through pt_mujoco: generated model, camera plugin, compressed image
pt_control's launch builds the MJCF with pt_mujoco at launch time (mujoco_scene selects the
scene), loads the CameraPlugin config from pt_mujoco at the real 30 Hz pipeline rate, and adds
the compressed image republisher and the optical-frame static TF. pt_bringup's gui argument is
now mujoco_gui and defaults to headless. The MJCF library no longer carries its own scene.

Co-Authored-By: Claude Sonnet 5 <noreply@anthropic.com>

File: pt_description/urdf/pantilt.control.xacro (robot description, xacro)
@@ -27,8 +27,7 @@
        used when the <gazebo> plugin below is actually instantiated (i.e. in sim). -->
   <xacro:arg name="simulation_controllers" default=""/>
-  <!-- mujoco mode only: path to the xacro-generated MJCF scene (pt_mujoco/mjcf/
-       pantilt.mjcf.xacro, xacro-processed at launch time with pantilt_config picking the
-       pt100/pt101 mesh variant - see pt_control/launch/pantilt.launch.py) and whether to
-       open the MuJoCo Simulate viewer window. -->
+  <!-- mujoco mode only: path to the MJCF generated by pt_mujoco's build_mujoco_models (see
+       pt_control/launch/pantilt.launch.py; pantilt_config picks the pt100/pt101 variant) and
+       whether to open the MuJoCo Simulate viewer window. -->
   <xacro:arg name="mujoco_model" default=""/>
   <xacro:arg name="mujoco_headless" default="false"/>

File: pt_mujoco/mjcf/pantilt.mjcf.xacro (robot description, xacro)
@@ -1,17 +1,9 @@
 <?xml version="1.0"?>
-<!-- Parametric PT100/PT101 MJCF assembly (mujoco_ros2_control equivalent of
-     pantilt.module.xacro + pantilt.urdf.xacro): defines the pantilt_body macro, selected by
-     pantilt_config, and when standalone:=true (default) invokes it in worldbody plus a
-     floor/lighting scene.
-     Standalone: xacro pantilt.mjcf.xacro pantilt_config:=pt101 > /tmp/pantilt.xml
-     pt_control/launch/pantilt.launch.py runs the same command at launch time.
-     Embedded (lekiwi_ros2's base_pantilt.mjcf.xacro): the includer declares its own
-     standalone:=false BEFORE including this file, which wins - xacro takes the first
-     <xacro:arg> declaration of a given name, later ones are ignored - and invokes
-     pantilt_body itself at its own mount point. Without this the worldbody+scene block
-     below would duplicate the whole assembly. -->
+<!-- Parametric PT100/PT101 MJCF library (mujoco_ros2_control equivalent of pantilt.module.xacro):
+     defines the pantilt_body macro, selected by pantilt_config. pt.mjcf.xacro fixes it to the
+     world for standalone use; scenes come from mjcf/scenes and are composed by
+     build_mujoco_models.py, which also syncs the numbers below from the URDF. -->
 <mujoco xmlns:xacro="http://www.ros.org/wiki/xacro" model="pantilt">
   <xacro:arg name="pantilt_config" default="pt101"/>
-  <xacro:arg name="standalone" default="true"/>
   <xacro:property name="pantilt_config" value="$(arg pantilt_config)"/>
   <!-- xacro:include, not a plain <include> - pantilt_shared.xml's mesh paths use $(find),
@@ -81,29 +73,3 @@
     </body>
   </xacro:macro>
-  <!-- Compares $(arg standalone) directly, not via a bridged <xacro:property> - xacro
-       auto-coerces "true"/"false" property values to Python bool, breaking a naive
-       string comparison. -->
-  <xacro:if value="${'$(arg standalone)' == 'true'}">
-    <worldbody>
-      <xacro:pantilt_body/>
-    </worldbody>
-    <statistic center="0.05 0 0.1" extent="0.4"/>
-    <visual>
-      <headlight diffuse="0.6 0.6 0.6" ambient="0.3 0.3 0.3" specular="0 0 0"/>
-      <rgba haze="0.15 0.25 0.35 1"/>
-      <global azimuth="45" elevation="-20"/>
-    </visual>
-    <asset>
-      <texture type="skybox" builtin="gradient" rgb1="0.3 0.5 0.7" rgb2="0 0 0" width="512" height="3072"/>
-      <texture type="2d" name="groundplane" builtin="checker" mark="edge" rgb1="0.2 0.3 0.4" rgb2="0.1 0.2 0.3"
-        markrgb="0.8 0.8 0.8" width="300" height="300"/>
-      <material name="groundplane" texture="groundplane" texuniform="true" texrepeat="5 5" reflectance="0.2"/>
-    </asset>
-    <worldbody>
-      <light pos="0 0 1.5" dir="0 0 -1" directional="true"/>
-      <!-- Non-colliding - this is a bracket meant to bolt to something, not a floor-standing
-           part; its base mesh legitimately extends below the mount plane. -->
-      <geom name="floor" size="0 0 0.05" type="plane" material="groundplane" contype="0" conaffinity="0"/>
-    </worldbody>
-  </xacro:if>
 </mujoco>

File: pt_mujoco/mjcf/pt.mjcf.xacro (robot description, xacro)
@@ -6,7 +6,4 @@
 <mujoco xmlns:xacro="http://www.ros.org/wiki/xacro" model="pantilt">
   <xacro:arg name="pantilt_config" default="pt101"/>
-  <!-- Declared BEFORE the include (xacro keeps the first declaration) so the library does not
-       add its own worldbody and scene on top of this one. -->
-  <xacro:arg name="standalone" default="false"/>
   <xacro:include filename="$(find pt_mujoco)/mjcf/pantilt.mjcf.xacro"/>
   <worldbody>

Commit message: Own the controller config, unlimited servo velocity in sim, e-stop and depth-to-scan wiring
Move pantilt_controller into pt_control/config/pantilt_controller.yaml, use the 1e6 velocity sentinel for mujoco as for real, stiffen the simulated end stops, load estop_mujoco_plugin, and add the /oak/scan depth slice to the sim.

Co-Authored-By: Claude Sonnet 5 <noreply@anthropic.com>

File: pt_description/urdf/pantilt.control.xacro (robot description, xacro)
@@ -45,5 +45,5 @@
        pantilt_max_velocity_rads duplicates pantilt_joints' own local computation
        (pantilt.joints.xacro) - only used by module.xacro's gazebo-mode <limit velocity>,
-       real mode keeps velocity="1e6" (see module.xacro's comment on why) regardless. -->
+       real and mujoco modes keep velocity="1e6" (see module.xacro's comment on why) regardless. -->
   <!-- This project runs the 12V STS3215 variant: 30 kgf*cm stall torque per Feetech's
        datasheet for that voltage option (not the 7.4V/19.5 kgf*cm variant used by stock

File: pt_description/urdf/pantilt.module.xacro (robot description, xacro)
@@ -94,8 +94,9 @@
       </collision>
     </link>
-    <!-- real mode: velocity="1e6" (unreachable) disables JointSaturationLimiter's clipping,
-         since joy_teleop's absolute position jumps would otherwise trip spurious limit
-         errors. gazebo mode: uses the real computed ceiling instead, since GazeboSimSystem
-         actually enforces this limit on the simulated joint. -->
+    <!-- real and mujoco modes: velocity="1e6" (unreachable) disables JointSaturationLimiter's
+         clipping, since joy_teleop's absolute position jumps would otherwise trip spurious limit
+         errors (MuJoCo does not need the limit: its servo model already bounds the motion).
+         gazebo mode: uses the real computed ceiling instead, since GazeboSimSystem actually
+         enforces this limit on the simulated joint. -->
     <!-- Shoulder-pan joint (revolute; was "pan_joint") -->
     <joint name="shoulder_pan_joint" type="revolute">
@@ -104,5 +105,5 @@
       <origin xyz="${shoulder_pan_x} 0 ${shoulder_pan_z}" rpy="0 0 0"/>
       <axis xyz="0 0 1"/>
-      <limit lower="${shoulder_pan_lower}" upper="${shoulder_pan_upper}" effort="${max_torque_nm}" velocity="${1e6 if '$(arg ros2_control_hardware_type)' == 'real' else pantilt_max_velocity_rads}"/>
+      <limit lower="${shoulder_pan_lower}" upper="${shoulder_pan_upper}" effort="${max_torque_nm}" velocity="${1e6 if '$(arg ros2_control_hardware_type)' in ('real', 'mujoco') else pantilt_max_velocity_rads}"/>
     </joint>
     <!-- Tilt joint (revolute) -->
@@ -112,5 +113,5 @@
       <origin xyz="${tilt_joint_x} 0 ${tilt_joint_z}" rpy="${tilt_joint_rx} ${tilt_joint_ry} 0"/>
       <axis xyz="0 0 -1"/>
-      <limit lower="${tilt_joint_lower}" upper="${tilt_joint_upper}" effort="${max_torque_nm}" velocity="${1e6 if '$(arg ros2_control_hardware_type)' == 'real' else pantilt_max_velocity_rads}"/>
+      <limit lower="${tilt_joint_lower}" upper="${tilt_joint_upper}" effort="${max_torque_nm}" velocity="${1e6 if '$(arg ros2_control_hardware_type)' in ('real', 'mujoco') else pantilt_max_velocity_rads}"/>
     </joint>
     <!-- OAK-D-S2 Camera + IMU -->

File: pt_mujoco/mjcf/sts3215.mjcf.xacro (robot description, xacro)
@@ -13,5 +13,9 @@
          deprecated tool). kp/error_gain/max_pwm=32/0.166/0.97 are STS3215Actuator's firmware
          constants (fixed across supply voltages); vin=12 for this identified variant. -->
-    <joint damping="1.057835" frictionloss="0.195871" armature="0.032460"/>
+    <!-- solreflimit/solimplimit: stiff end stops. With MuJoCo's default soft limit a full-speed jump to
+         a limit penetrates it by ~0.01 rad, and ros2_control's limiter treats a measured position
+         beyond the URDF limit as a hardware fault and deactivates the controller. -->
+    <joint damping="1.057835" frictionloss="0.195871" armature="0.032460"
+           solreflimit="0.004 1" solimplimit="0.99 0.999 0.001 0.5 2"/>
     <position kp="42.911886" kv="0.0" forcerange="-8.537717 8.537717"/>
     <!-- so_arm_mujoco's copy also nests visual/collision geom sub-classes for its own STS3215
