Commit message: Add pt_mujoco, own the controller config, package READMEs and single-quote style (#3)
* Drop the MuJoCo camera GLFW note from the simulation section

The camera now works in sim through the CameraPlugin with headless EGL
rendering (see lekiwi_mujoco), so the not-working explanation no longer applies.

Co-Authored-By: Claude Sonnet 5 <noreply@anthropic.com>

* Add pt_mujoco package skeleton

Co-Authored-By: Claude Sonnet 5 <noreply@anthropic.com>

* Move the MJCF from pt_description into pt_mujoco

The MJCF, its tests and a bundled flat scene now live in pt_mujoco; pt_description keeps the
URDF and meshes. pt_control locates the MJCF through pt_mujoco.

Co-Authored-By: Claude Sonnet 5 <noreply@anthropic.com>

* pt_mujoco: standalone URDF-driven builder, simulation, viewer, benchmark and tests

The builder expands pt_description's URDF and syncs frames, mesh origins, inertias, actuator
effort and limits from it (replacing the stale tilt-joint height in the MJCF), then composes
the payload with a bundled flat scene. pt100 and pt101 snapshots are regenerated by it.

Co-Authored-By: Claude Sonnet 5 <noreply@anthropic.com>

* Run the pan-tilt sim through pt_mujoco: generated model, camera plugin, compressed image

pt_control's launch builds the MJCF with pt_mujoco at launch time (mujoco_scene selects the
scene), loads the CameraPlugin config from pt_mujoco at the real 30 Hz pipeline rate, and adds
the compressed image republisher and the optical-frame static TF. pt_bringup's gui argument is
now mujoco_gui and defaults to headless. The MJCF library no longer carries its own scene.

Co-Authored-By: Claude Sonnet 5 <noreply@anthropic.com>

* pt_mujoco: build_payload_spec builds the payload from any host URDF

A host robot passes its own expanded URDF and joint limits and attaches the returned spec at its
mount frame; the standalone builder now goes through the same function. The payload's inertia sync
is limited to its own links so a larger URDF works, and physics options are left to the composed
model instead of being set on the payload spec.

Co-Authored-By: Claude Sonnet 5 <noreply@anthropic.com>

* Document pt_mujoco and add it to CI

README: pt_mujoco package, mujoco_gui/mujoco_scene arguments, simulated camera, updated tree and
Simulation section. CI builds pt_mujoco, runs the pytest suites, and adds a Linux/macOS/Windows
MuJoCo job.

Co-Authored-By: Claude Sonnet 5 <noreply@anthropic.com>

* pt_mujoco: use the BAM-identified STS3215 profile for the pan and tilt servos

Adds sts3215.mjcf.xacro (class pt_sts3215, distinct from lekiwi's sts3215 so both can be composed)
and applies its gain, damping, armature and friction at build time like the wheels. The step
response settles in about 0.3 s with 4% (pan) to 8% (tilt) overshoot instead of 0.55 s with none.

Co-Authored-By: Claude Sonnet 5 <noreply@anthropic.com>

* pan-tilt: slow, smooth servo profile (65/50/0) is the module's own default

pantilt.joints.xacro's internal_* macro defaults are now 65/50/0 (near the STS3215 firmware's
own ~68/~50/1) instead of 254/254/100, which makes the pan-tilt accelerate fast enough to crash the
Pi. pt_control's urdf_config.yaml sets them explicitly so they can be tuned, and pt_control's launch
passes them through pantilt.control.xacro. Prebuilt URDFs are regenerated and tests pin the values.

Co-Authored-By: Claude Sonnet 5 <noreply@anthropic.com>

* Own the controller config, unlimited servo velocity in sim, e-stop and depth-to-scan wiring

Move pantilt_controller into pt_control/config/pantilt_controller.yaml, use the 1e6 velocity sentinel for mujoco as for real, stiffen the simulated end stops, load estop_mujoco_plugin, and add the /oak/scan depth slice to the sim.

Co-Authored-By: Claude Sonnet 5 <noreply@anthropic.com>

* Load the renamed mujoco_ros2_plugins package

Co-Authored-By: Claude Sonnet 5 <noreply@anthropic.com>

* Link the mujoco_ros2_plugins repository

Co-Authored-By: Claude Sonnet 5 <noreply@anthropic.com>

* Rewrite the README: shorter, one path from install to configuration to simulation

Co-Authored-By: Claude Sonnet 5 <noreply@anthropic.com>

* README: list the files users may edit

Co-Authored-By: Claude Sonnet 5 <noreply@anthropic.com>

* pt_mujoco README: shorter and current; correct the joint_limits description

Co-Authored-By: Claude Sonnet 5 <noreply@anthropic.com>

* Shorten comments and docstrings

Co-Authored-By: Claude Sonnet 5 <noreply@anthropic.com>

* Trim comments and docstrings to one line, refresh package.xml files, drop test_without_ros

Co-Authored-By: Claude Sonnet 5 <noreply@anthropic.com>

* Add a pt_description README

Co-Authored-By: Claude Sonnet 5 <noreply@anthropic.com>

* Add a pt_control README and fix the diagnostics default in the main README

Co-Authored-By: Claude Sonnet 5 <noreply@anthropic.com>

* Add a pt_bringup README

Co-Authored-By: Claude Sonnet 5 <noreply@anthropic.com>

* pt_bringup README: correct the CI note

Co-Authored-By: Claude Sonnet 5 <noreply@anthropic.com>

* Give the four package READMEs one structure

Co-Authored-By: Claude Sonnet 5 <noreply@anthropic.com>

* READMEs: drop sections with nothing to say

Co-Authored-By: Claude Sonnet 5 <noreply@anthropic.com>

* Top-level README: same structure as the package READMEs

Co-Authored-By: Claude Sonnet 5 <noreply@anthropic.com>

* Shorten the ruff config comment and ignore tool caches

Co-Authored-By: Claude Sonnet 5 <noreply@anthropic.com>

* Use single quotes across all Python files and enforce them with ruff

Co-Authored-By: Claude Sonnet 5 <noreply@anthropic.com>

* CI: drop the Windows job

Co-Authored-By: Claude Sonnet 5 <noreply@anthropic.com>

* Address review: validate mujoco_gui, clean up the generated MJCF, declare the plugin provider, report an unsettled response, fix the pip path

Co-Authored-By: Claude Sonnet 5 <noreply@anthropic.com>

---------

Co-authored-by: Claude Sonnet 5 <noreply@anthropic.com>

File: pt_description/urdf/pantilt.control.xacro (robot description, xacro)
@@ -8,27 +8,16 @@
   <xacro:arg name="sts3215_max_vel_steps" default="3400"/>   <!-- STS3215=3400, STS3032=2900, STS3235=3400 -->
   <xacro:arg name="proportional_vel_max"   default="0"/>      <!-- [0-max_velocity_steps]; 0 = each joint uses commanded velocity -->
-  <!-- Motor IDs, step-centering, and joint limits are NOT xacro:args here - they're
-       physical-calibration constants for this mechanism (motor wiring, servo centering),
-       not per-deployment connection settings, so pantilt.joints.xacro's macro defaults are
-       their single source of truth (same convention as so101.control.xacro/so100.control.xacro
-       in so_arm_ros2, which hardcode motor IDs/joint limits as fixed xacro:property values
-       rather than sourcing them from an external launch-time YAML). A host embedding this
-       mechanism on a shared bus (e.g. lekiwi_ros2's base_pantilt.control.xacro) can still
-       override any of pantilt_joints' macro params explicitly if it ever needs different
-       values - see pantilt.joints.xacro. -->
+  <!-- Servo EEPROM profile (0-254), defaults match pantilt.joints.xacro; urdf_config.yaml sets them for tuning -->
+  <xacro:arg name="internal_max_vel"       default="65"/>
+  <xacro:arg name="internal_max_acc"       default="50"/>
+  <xacro:arg name="internal_acc_coeff"     default="0"/>
+  <!-- Motor IDs, centres and joint limits are calibration constants: pantilt.joints.xacro macro defaults hold them -->
   <!-- Simulation -->
-  <!-- "real" (default) keeps the STS3215 serial hardware plugin below unchanged.
-       "gazebo" swaps the <hardware> plugin for gz_ros2_control/GazeboSimSystem.
-       "mujoco" swaps it for mujoco_ros2_control/MujocoSystemInterface.
-       Both implement the same SystemInterface contract - the joints and controllers stay
-       identical in all three cases. -->
+  <!-- Hardware plugin: real (STS3215, default), gazebo or mujoco; joints and controllers are identical -->
   <xacro:arg name="ros2_control_hardware_type" default="real"/>
   <!-- Path to the controllers YAML the embedded controller_manager should load; only
        used when the <gazebo> plugin below is actually instantiated (i.e. in sim). -->
   <xacro:arg name="simulation_controllers" default=""/>
-  <!-- mujoco mode only: path to the xacro-generated MJCF scene (pt_description/mjcf/
-       pantilt.mjcf.xacro, xacro-processed at launch time with pantilt_config picking the
-       pt100/pt101 mesh variant - see pt_control/launch/pantilt.launch.py) and whether to
-       open the MuJoCo Simulate viewer window. -->
+  <!-- mujoco only: generated MJCF path and whether to open the viewer -->
   <xacro:arg name="mujoco_model" default=""/>
   <xacro:arg name="mujoco_headless" default="false"/>
@@ -36,12 +25,6 @@
        because pantilt_joints (called below) writes it per joint as max_velocity_steps. -->
   <xacro:property name="sts3215_max_vel_steps" value="$(arg sts3215_max_vel_steps)"/>
-  <!-- Torque limit as a top-level property — required by pantilt.module.xacro for the URDF
-       <limit> elements on the revolute joints.
-       pantilt_max_velocity_rads duplicates pantilt_joints' own local computation
-       (pantilt.joints.xacro) - only used by module.xacro's gazebo-mode <limit velocity>,
-       real mode keeps velocity="1e6" (see module.xacro's comment on why) regardless. -->
-  <!-- This project runs the 12V STS3215 variant: 30 kgf*cm stall torque per Feetech's
-       datasheet for that voltage option (not the 7.4V/19.5 kgf*cm variant used by stock
-       SO-ARM100/101). -->
+  <!-- Torque limit for the module's revolute joint <limit> elements -->
+  <!-- 12V STS3215: 30 kgf*cm stall torque -->
   <xacro:property name="max_torque_nm"    value="2.942"/>  <!-- N⋅m (30 kgf⋅cm @ 12V) -->
   <xacro:property name="pantilt_max_velocity_steps" value="${int(sts3215_max_vel_steps * 0.85)}"/>
@@ -72,5 +55,8 @@
     <xacro:pantilt_joints
         sts3215_max_vel_steps="${sts3215_max_vel_steps}"
-        ros2_control_hardware_type="$(arg ros2_control_hardware_type)"/>
+        ros2_control_hardware_type="$(arg ros2_control_hardware_type)"
+        internal_max_vel="$(arg internal_max_vel)"
+        internal_max_acc="$(arg internal_max_acc)"
+        internal_acc_coeff="$(arg internal_acc_coeff)"/>
   </ros2_control>
 </robot>

File: pt_description/urdf/pantilt.joints.xacro (robot description, xacro)
@@ -1,21 +1,5 @@
 <?xml version="1.0"?>
 <robot xmlns:xacro="http://www.ros.org/wiki/xacro">
-  <!--
-    pantilt_joints macro — ros2_control joint declarations for the PT100 pan-tilt.
-    Intended for embedding into a host robot's <ros2_control> block when the
-    PT100 shares the host's serial bus (and therefore its hardware interface).
-    For standalone use, pantilt.control.xacro wraps this in its own <ros2_control>
-    block with the STSHardwareInterface plugin.
-    Params:
-      shoulder_pan_motor_id — STS3215 motor ID for pan axis
-      tilt_motor_id         — STS3215 motor ID for tilt axis
-      shoulder_pan_center_steps — raw step value (0–4095) for pan centre position
-      tilt_center_steps     — raw step value (0–4095) for tilt centre position
-      sts3215_max_vel_steps — motor's max velocity in steps/s, model-dependent;
-                               written per joint as max_velocity_steps
-      internal_max_vel      — EEPROM VMax cap (addr 84), written per joint
-      internal_max_acc      — EEPROM AMax cap (addr 85), written per joint
-      internal_acc_coeff    — EEPROM KAcc coefficient (addr 86), written per joint
-  -->
+  <!-- pantilt_joints: ros2_control joints for a host's shared-bus block; defaults are the mechanism's calibration and the slow 65/50/0 servo profile -->
   <xacro:macro name="pantilt_joints" params="
       shoulder_pan_motor_id:=1
@@ -28,7 +12,7 @@
       tilt_joint_lower:=-1.5708
       tilt_joint_upper:=1.5708
-      internal_max_vel:=254
-      internal_max_acc:=254
-      internal_acc_coeff:=100
+      internal_max_vel:=65
+      internal_max_acc:=50
+      internal_acc_coeff:=0
       ros2_control_hardware_type:=real">
     <!-- 85% of hardware max — 15% safety margin; motor firmware handles profiling -->
@@ -52,7 +36,5 @@
       <state_interface name="velocity"/>
       <state_interface name="effort"/>
-      <!-- Real-hardware-only telemetry: neither gz_ros2_control/GazeboSimSystem nor
-           mujoco_ros2_control/MujocoSystemInterface know position/velocity/effort-only
-           joints, and simulated joints have no real telemetry for these. -->
+      <!-- Real hardware only: sim joints have no such telemetry -->
       <xacro:if value="${ros2_control_hardware_type == 'real'}">
         <state_interface name="voltage"/>
@@ -79,7 +61,5 @@
       <state_interface name="velocity"/>
       <state_interface name="effort"/>
-      <!-- Real-hardware-only telemetry: neither gz_ros2_control/GazeboSimSystem nor
-           mujoco_ros2_control/MujocoSystemInterface know position/velocity/effort-only
-           joints, and simulated joints have no real telemetry for these. -->
+      <!-- Real hardware only: sim joints have no such telemetry -->
       <xacro:if value="${ros2_control_hardware_type == 'real'}">
         <state_interface name="voltage"/>

File: pt_description/urdf/pantilt.module.xacro (robot description, xacro)
@@ -94,8 +94,5 @@
       </collision>
     </link>
-    <!-- real mode: velocity="1e6" (unreachable) disables JointSaturationLimiter's clipping,
-         since joy_teleop's absolute position jumps would otherwise trip spurious limit
-         errors. gazebo mode: uses the real computed ceiling instead, since GazeboSimSystem
-         actually enforces this limit on the simulated joint. -->
+    <!-- real/mujoco: 1e6 avoids spurious limit trips on joystick jumps; gazebo enforces the real ceiling -->
     <!-- Shoulder-pan joint (revolute; was "pan_joint") -->
     <joint name="shoulder_pan_joint" type="revolute">
@@ -104,5 +101,5 @@
       <origin xyz="${shoulder_pan_x} 0 ${shoulder_pan_z}" rpy="0 0 0"/>
       <axis xyz="0 0 1"/>
-      <limit lower="${shoulder_pan_lower}" upper="${shoulder_pan_upper}" effort="${max_torque_nm}" velocity="${1e6 if '$(arg ros2_control_hardware_type)' == 'real' else pantilt_max_velocity_rads}"/>
+      <limit lower="${shoulder_pan_lower}" upper="${shoulder_pan_upper}" effort="${max_torque_nm}" velocity="${1e6 if '$(arg ros2_control_hardware_type)' in ('real', 'mujoco') else pantilt_max_velocity_rads}"/>
     </joint>
     <!-- Tilt joint (revolute) -->
@@ -112,5 +109,5 @@
       <origin xyz="${tilt_joint_x} 0 ${tilt_joint_z}" rpy="${tilt_joint_rx} ${tilt_joint_ry} 0"/>
       <axis xyz="0 0 -1"/>
-      <limit lower="${tilt_joint_lower}" upper="${tilt_joint_upper}" effort="${max_torque_nm}" velocity="${1e6 if '$(arg ros2_control_hardware_type)' == 'real' else pantilt_max_velocity_rads}"/>
+      <limit lower="${tilt_joint_lower}" upper="${tilt_joint_upper}" effort="${max_torque_nm}" velocity="${1e6 if '$(arg ros2_control_hardware_type)' in ('real', 'mujoco') else pantilt_max_velocity_rads}"/>
     </joint>
     <!-- OAK-D-S2 Camera + IMU -->
