Commit message: Add Gemini 2 camera variants and aligned pan-tilt simulation assets

File: pt_description/urdf/camera.module.xacro (robot description, xacro)
@@ -1,18 +1,18 @@
 <?xml version="1.0"?>
-<robot name="depthai_camera"
+<robot name="camera"
 	xmlns:xacro="http://ros.org/wiki/xacro">
-	<!-- OAK-D S2 camera macro shared by pt100/pt101, with r/g/b/a mesh colour parameters -->
-	<xacro:macro name="oakd_s2_camera"
+	<!-- Camera macro shared by PT100/PT101 and OAK-D S2/Gemini 2, with r/g/b/a mesh colour parameters -->
+	<xacro:macro name="camera"
 		params="camera_name parent base_frame
 											   cam_pos_x cam_pos_y cam_pos_z
 											   cam_roll cam_pitch cam_yaw
 											   r:=0.1 g:=0.1 b:=0.1 a:=1.0 simulation:=false
-											   imu_frame:=oak_imu_frame">
+											   imu_frame:=oak_imu_frame mesh_file:=oakd_s2.stl mesh_yaw:=0">
 		<!-- File prefix for mesh location -->
 		<xacro:if value="${simulation}">
-			<xacro:property name="mesh_path" value="file://$(find pt_description)/meshes/oakd_s2.stl" />
+			<xacro:property name="mesh_path" value="file://$(find pt_description)/meshes/${mesh_file}" />
 		</xacro:if>
 		<xacro:unless value="${simulation}">
-			<xacro:property name="mesh_path" value="package://pt_description/meshes/oakd_s2.stl" />
+			<xacro:property name="mesh_path" value="package://pt_description/meshes/${mesh_file}" />
 		</xacro:unless>
 		<!-- base_link of the sensor-->
@@ -35,9 +35,9 @@
 		<link name="${camera_name}_model_origin">
 			<visual>
-				<origin xyz="0 0 0" rpy="0 0 0" />
+				<origin xyz="0 0 0" rpy="0 0 ${mesh_yaw}" />
 				<geometry>
 					<mesh filename="${mesh_path}" />
 				</geometry>
-				<material name="mat">
+				<material name="camera_charcoal">
 					<color rgba="${r} ${g} ${b} ${a}" />
 				</material>

File: pt_description/urdf/pantilt.common.xacro (robot description, xacro)
@@ -8,4 +8,9 @@
   <xacro:arg name="pantilt_config" default="pt101"/>
   <xacro:property name="pantilt_config" value="$(arg pantilt_config)"/>
+  <!-- Camera choice is independent of the pan/tilt body variant. -->
+  <xacro:arg name="camera_config" default="oakd_s2"/>
+  <xacro:property name="camera_config" value="$(arg camera_config)"/>
+  <xacro:property name="camera_mesh" value="${dict(oakd_s2='oakd_s2.stl', gemini2='gemini2.stl')[camera_config]}"/>
+  <xacro:property name="tilt_camera_mesh" value="${dict(oakd_s2='tilt_joint_oakd_s2.stl', gemini2='tilt_joint_gemini2.stl')[camera_config]}"/>
   <!-- Pantilt base visual compensation / mount rotation (rad) -->
   <xacro:property name="pantilt_offset_rz" value="${pi/2}"/>
@@ -48,15 +53,26 @@
   <xacro:property name="tilt_visual_y" value="${shoulder_pan_x + tilt_joint_x}"/>
   <xacro:property name="tilt_visual_z" value="-0.0002"/>
-  <!-- OAK-D-S2 camera mount offset (in tilt_link frame) -->
-  <xacro:property name="oak_pos_x" value="-0.0306"/>
-  <xacro:property name="oak_pos_y" value="-0.012165"/>
-  <!-- OAK-D-S2 camera mount orientation (in tilt_link frame) -->
-  <xacro:property name="oak_roll" value="${-pi/2}"/>
-  <xacro:property name="oak_yaw"  value="${-pi/2}"/>
-  <!-- OAK-D-S2 IMU offset (relative to oak frame) -->
-  <xacro:property name="oak_imu_x" value="-0.008"/>
-  <xacro:property name="oak_imu_y" value="-0.037945"/>
-  <xacro:property name="oak_imu_z" value="-0.00079"/>
-  <xacro:property name="oak_imu_r" value="${pi}"/>
-  <xacro:property name="oak_imu_p" value="${pi/2}"/>
+  <!-- Camera mount offset (in tilt_link frame) -->
+  <xacro:property name="camera_pos_x" value="-0.0306"/>
+  <xacro:property name="camera_pos_y" value="-0.012165"/>
+  <xacro:property name="camera_pos_z" value="0"/>
+  <!-- Gemini rear face z=-18.65 mm seats on mount z=64.0441 mm in mesh/world X.
+       Required camera origin X=82.6941 mm; tilt origin X=75.8 mm, local Y=-world X. -->
+  <xacro:if value="${camera_config == 'gemini2'}">
+    <xacro:property name="camera_pos_y" value="-0.0068941"/>
+    <!-- Mount inner faces: -18.1/+18.75 mm in STL X; motor faces: -18.3/+18.1 mm.
+         Offset -0.425 mm centers the 36.85 mm opening on the 36.4 mm motor span,
+         leaving 0.225 mm per side. Shift the camera by the same additional -0.225 mm. -->
+    <xacro:property name="tilt_visual_z" value="-0.000425"/>
+    <xacro:property name="camera_pos_z" value="-0.000225"/>
+  </xacro:if>
+  <!-- Camera mount orientation (in tilt_link frame) -->
+  <xacro:property name="camera_roll" value="${-pi/2}"/>
+  <xacro:property name="camera_yaw"  value="${-pi/2}"/>
+  <!-- Compatibility IMU offset (OAK calibration) (relative to oak frame) -->
+  <xacro:property name="camera_imu_x" value="-0.008"/>
+  <xacro:property name="camera_imu_y" value="-0.037945"/>
+  <xacro:property name="camera_imu_z" value="-0.00079"/>
+  <xacro:property name="camera_imu_r" value="${pi}"/>
+  <xacro:property name="camera_imu_p" value="${pi/2}"/>
 </robot>

File: pt_description/urdf/pantilt.module.xacro (robot description, xacro)
@@ -2,5 +2,5 @@
 <robot xmlns:xacro="http://www.ros.org/wiki/xacro">
   <xacro:include filename="$(find pt_description)/urdf/pantilt.common.xacro"/>
-  <xacro:include filename="$(find pt_description)/urdf/oakd_s2.module.xacro"/>
+  <xacro:include filename="$(find pt_description)/urdf/camera.module.xacro"/>
   <xacro:macro name="pantilt_module" params="parent *origin">
     <!-- Material definitions (referenced by links below) -->
@@ -83,5 +83,5 @@
         <origin xyz="${tilt_visual_x} ${tilt_visual_y} ${tilt_visual_z}" rpy="${tilt_offset_rx} ${tilt_offset_ry} 0"/>
         <geometry>
-          <mesh filename="package://pt_description/meshes/tilt_joint_oakd_s2.stl"/>
+          <mesh filename="package://pt_description/meshes/${tilt_camera_mesh}"/>
         </geometry>
         <material name="light_grey"/>
@@ -90,5 +90,5 @@
         <origin xyz="${tilt_visual_x} ${tilt_visual_y} ${tilt_visual_z}" rpy="${tilt_offset_rx} ${tilt_offset_ry} 0"/>
         <geometry>
-          <mesh filename="package://pt_description/meshes/tilt_joint_oakd_s2.stl"/>
+          <mesh filename="package://pt_description/meshes/${tilt_camera_mesh}"/>
         </geometry>
       </collision>
@@ -111,11 +111,13 @@
       <limit lower="${tilt_joint_lower}" upper="${tilt_joint_upper}" effort="${max_torque_nm}" velocity="${1e6 if '$(arg ros2_control_hardware_type)' in ('real', 'mujoco') else pantilt_max_velocity_rads}"/>
     </joint>
-    <!-- OAK-D-S2 Camera + IMU -->
-    <xacro:oakd_s2_camera
+    <!-- Selected camera mesh + compatibility camera/IMU frames -->
+    <xacro:camera
+      mesh_file="${camera_mesh}"
+      mesh_yaw="${pi if camera_config == 'gemini2' else 0}"
       camera_name="oak_link"
       base_frame="oak_link"
       parent="tilt_link"
-      cam_pos_x="${oak_pos_x}" cam_pos_y="${oak_pos_y}" cam_pos_z="0"
-      cam_roll="${oak_roll}" cam_pitch="0" cam_yaw="${oak_yaw}"
+      cam_pos_x="${camera_pos_x}" cam_pos_y="${camera_pos_y}" cam_pos_z="${camera_pos_z}"
+      cam_roll="${camera_roll}" cam_pitch="0" cam_yaw="${camera_yaw}"
       r="${charcoal_rgb}" g="${charcoal_rgb}" b="${charcoal_rgb}" a="1.0"
       imu_frame="oak_imu_frame"/>

File: pt_description/urdf/pt101_gemini2.urdf (robot description, URDF)
Before this commit: robot pantilt, 7 links, 6 joints
Links:
- link oak_link_model_origin: geometry visual mesh filename=../meshes/gemini2.stl
- link tilt_link: geometry collision mesh filename=../meshes/tilt_joint_gemini2.stl; visual mesh filename=../meshes/tilt_joint_gemini2.stl
Joints:
- joint oak_link_center_joint: origin xyz=-0.0306 -0.012165 0 rpy=-1.5707963267948966 0 -1.5707963267948966 -> xyz=-0.0306 -0.0068941 -0.000225 rpy=-1.5707963267948966 0 -1.5707963267948966

File: pt_description/urdf/pt101_oakd_s2.urdf (robot description, URDF)
Before this commit: robot pantilt, 7 links, 6 joints
Links:
- link pantilt_base_link: geometry collision mesh filename=../meshes/pantilt_base_101.stl; visual mesh filename=../meshes/pan_motor.stl
- link shoulder_link: geometry collision mesh filename=../meshes/pan_joint_101.stl; visual mesh filename=../meshes/pan_joint_101.stl

File: pt_mujoco/mjcf/pantilt.mjcf.xacro (robot description, xacro)
@@ -2,4 +2,6 @@
 <!-- Parametric PT100/PT101 MJCF (pantilt_body macro, selected by pantilt_config); build_mujoco_models.py syncs the numbers from the URDF -->
 <mujoco xmlns:xacro="http://www.ros.org/wiki/xacro" model="pantilt">
+  <xacro:arg name="camera_config" default="oakd_s2"/>
+  <xacro:property name="camera_config" value="$(arg camera_config)"/>
   <xacro:arg name="pantilt_config" default="pt101"/>
   <xacro:property name="pantilt_config" value="$(arg pantilt_config)"/>
@@ -51,5 +53,5 @@
         <geom mesh="shoulder_link_mesh" class="collision"
               pos="${shoulder_link_geom_pos}" quat="${shoulder_link_geom_quat}"/>
-        <include file="$(find pt_mujoco)/mjcf/oakd_s2_subtree.xml"/>
+        <include file="$(find pt_mujoco)/mjcf/${camera_config}_subtree.xml"/>
       </body>
     </body>
