Commit message: Fix Gemini2 and OAK-D camera frame orientation

File: pt_description/urdf/pantilt.common.xacro (robot description, xacro)
@@ -13,4 +13,6 @@
   <xacro:property name="camera_mesh" value="${dict(oakd_s2='oakd_s2.stl', gemini2='gemini2.stl')[camera_config]}"/>
   <xacro:property name="tilt_camera_mesh" value="${dict(oakd_s2='tilt_joint_oakd_s2.stl', gemini2='tilt_joint_gemini2.stl')[camera_config]}"/>
+  <xacro:property name="camera_base_frame" value="${'gemini2_link' if camera_config == 'gemini2' else 'oak_link'}"/>
+  <xacro:property name="camera_imu_frame" value="${'gemini2_imu_frame' if camera_config == 'gemini2' else 'oak_imu_frame'}"/>
   <!-- Pantilt base visual compensation / mount rotation (rad) -->
   <xacro:property name="pantilt_offset_rz" value="${pi/2}"/>
@@ -70,4 +72,8 @@
   <xacro:property name="camera_roll" value="${-pi/2}"/>
   <xacro:property name="camera_yaw"  value="${-pi/2}"/>
+  <!-- Gemini 2 is mounted upright (the OAK-D frame already absorbs its upside-down mount): +pi about its forward axis -->
+  <xacro:if value="${camera_config == 'gemini2'}">
+    <xacro:property name="camera_roll" value="${pi/2}"/>
+  </xacro:if>
   <!-- Compatibility IMU offset (OAK calibration) (relative to oak frame) -->
   <xacro:property name="camera_imu_x" value="-0.008"/>

File: pt_description/urdf/pantilt.module.xacro (robot description, xacro)
@@ -114,12 +114,12 @@
     <xacro:camera
       mesh_file="${camera_mesh}"
-      mesh_yaw="${pi if camera_config == 'gemini2' else 0}"
-      camera_name="oak_link"
-      base_frame="oak_link"
+      mesh_yaw="0"
+      camera_name="${camera_base_frame}"
+      base_frame="${camera_base_frame}"
       parent="tilt_link"
       cam_pos_x="${camera_pos_x}" cam_pos_y="${camera_pos_y}" cam_pos_z="${camera_pos_z}"
       cam_roll="${camera_roll}" cam_pitch="0" cam_yaw="${camera_yaw}"
       r="${charcoal_rgb}" g="${charcoal_rgb}" b="${charcoal_rgb}" a="1.0"
-      imu_frame="oak_imu_frame"/>
+      imu_frame="${camera_imu_frame}"/>
   </xacro:macro>
 </robot>

File: pt_description/urdf/pt100_gemini2.urdf (robot description, URDF)
Before this commit: robot pantilt, 7 links, 6 joints
Links:
- removed link oak_imu_frame
- removed link oak_link
- removed link oak_link_model_origin
- added link gemini2_imu_frame
- added link gemini2_link
- added link gemini2_link_model_origin; visual mesh filename=../meshes/gemini2.stl
Joints:
- removed joint oak_imu_frame_joint
- removed joint oak_link_center_joint
- removed joint oak_link_model_origin_joint
- added joint gemini2_imu_frame_joint: type fixed, parent gemini2_link, child gemini2_imu_frame, origin xyz=-0.008 -0.037945 -0.00079 rpy=3.141592653589793 1.5707963267948966 0
- added joint gemini2_link_center_joint: type fixed, parent tilt_link, child gemini2_link, origin xyz=-0.0306 -0.0068941 -0.000225 rpy=1.5707963267948966 0 -1.5707963267948966
- added joint gemini2_link_model_origin_joint: type fixed, parent gemini2_link, child gemini2_link_model_origin, origin xyz=0 0 0 rpy=1.5707963267948966 0 1.5707963267948966

File: pt_description/urdf/pt101_gemini2.urdf (robot description, URDF)
Before this commit: robot pantilt, 7 links, 6 joints
Links:
- removed link oak_imu_frame
- removed link oak_link
- removed link oak_link_model_origin
- added link gemini2_imu_frame
- added link gemini2_link
- added link gemini2_link_model_origin; visual mesh filename=../meshes/gemini2.stl
Joints:
- removed joint oak_imu_frame_joint
- removed joint oak_link_center_joint
- removed joint oak_link_model_origin_joint
- added joint gemini2_imu_frame_joint: type fixed, parent gemini2_link, child gemini2_imu_frame, origin xyz=-0.008 -0.037945 -0.00079 rpy=3.141592653589793 1.5707963267948966 0
- added joint gemini2_link_center_joint: type fixed, parent tilt_link, child gemini2_link, origin xyz=-0.0306 -0.0068941 -0.000225 rpy=1.5707963267948966 0 -1.5707963267948966
- added joint gemini2_link_model_origin_joint: type fixed, parent gemini2_link, child gemini2_link_model_origin, origin xyz=0 0 0 rpy=1.5707963267948966 0 1.5707963267948966
